Commit message: Gazebo Harmonic migration and adding sdf file for simulation with lidar and camera

File: ROS/osr_gazebo/urdf/gazebo.urdf.xacro (robot description, xacro)
@@ -3,5 +3,5 @@
   <ros2_control name="GazeboSystem" type="system">
     <hardware>
-      <plugin>gazebo_ros2_control/GazeboSystem</plugin>
+      <plugin>gz_ros2_control/GazeboSimSystem</plugin>
     </hardware>
     <joint name="middle_wheel_joint_left">
@@ -110,10 +110,32 @@
       <state_interface name="effort"/>
     </joint>
+    <joint name="rocker_bogie_joint_L_2">
+      <state_interface name="position"/>
+      <state_interface name="velocity"/>
+      <state_interface name="effort"/>
+    </joint>
+    <joint name="rocker_bogie_joint_R_2">
+      <state_interface name="position"/>
+      <state_interface name="velocity"/>
+      <state_interface name="effort"/>
+    </joint>
   </ros2_control>
   <gazebo>
-    <plugin filename="libgazebo_ros2_control.so" name="gazebo_ros2_control">
+    <plugin filename="gz_ros2_control-system" name="gz_ros2_control::GazeboSimROS2ControlPlugin">
       <parameters>$(find osr_gazebo)/config/controller_velocity.yaml</parameters>
     </plugin>
   </gazebo>
+  <gazebo>
+    <plugin filename="gz-sim-joint-state-publisher-system" name="gz::sim::systems::JointStatePublisher">
+      <topic>joint_states</topic>
+      <joint_name>rear_wheel_joint_right</joint_name>
+      <joint_name>rear_wheel_joint_left</joint_name>
+      <joint_name>middle_wheel_joint_right</joint_name>
+      <joint_name>middle_wheel_joint_left</joint_name>
+      <joint_name>front_wheel_joint_right</joint_name>
+      <joint_name>front_wheel_joint_left</joint_name>
+    </plugin>
+  </gazebo>
+<!--
     <gazebo reference="imu_link">
         <gravity>true</gravity>
@@ -123,5 +145,5 @@
         <visualize>true</visualize>
         <topic>"imu"</topic>
-        <plugin filename="libgazebo_ros_imu_sensor.so" name="imu_plugin">
+        <plugin filename="libgz_ros_imu_sensor.so" name="imu_plugin">
             <topicName>imu</topicName>
             <bodyName>imu_link</bodyName>
@@ -136,3 +158,4 @@
         </sensor>
     </gazebo>
+-->
 </robot>

File: ROS/osr_gazebo/urdf/osr.urdf.xacro (robot description, xacro)
@@ -14,8 +14,13 @@
     </material>
     <material name="brown">
-      <color rgba="0.5451 0.2706 0.0745 1"/>
+      <color rgba="0.5451 0.2706 0.0745 0.5"/>
+    </material>
+    <material name="red">
+        <color rgba="1 0 0 0.8"/>
     </material>
     <xacro:include filename="$(find osr_gazebo)/urdf/gazebo.urdf.xacro"/>
-    <xacro:include filename="$(find osr_gazebo)/urdf/insert_transmission.urdf.xacro"/>
+    <!-- <xacro:include filename="$(find osr_gazebo)/urdf/insert_transmission.urdf.xacro"/> -->
+    <xacro:include filename="$(find osr_gazebo)/urdf/lidar.urdf.xacro"/>
+    <xacro:include filename="$(find osr_gazebo)/urdf/camera.urdf.xacro"/>
     <link name="base_footprint"/>
     <link name="base_link">
@@ -420,4 +425,5 @@
         </joint>
     <link name="imu_link"></link>
+<!--
     <xacro:insert_velocity_transmission name="rear_wheel_joint_right"/>
     <xacro:insert_velocity_transmission name="rear_wheel_joint_left"/>
@@ -430,3 +436,4 @@
     <xacro:insert_position_transmission name="rear_wheel_joint_R"/>
     <xacro:insert_position_transmission name="rear_wheel_joint_L"/>
+-->
 </robot>
